Commit message: add trashcan stl corrected

File: src/iiwa_stack_examples/iiwa_tool/iiwa_tool_description/urdf/iiwa14_tool.urdf.xacro (robot description, xacro)
@@ -44,5 +44,5 @@
   <!-- <mesh filename="package://my_egg_sensor_desc/meshes/egg_50cm_1600.stl"/> -->
 	<!-- <mesh filename="package://iiwa_tool_description/meshes/visual/tool.stl"/> -->
-		<cylinder length="0.2550" radius="0.020"/>
+		<cylinder length="0.23" radius="0.020"/>
       </geometry>
       <material name="Grey"/>
@@ -53,5 +53,5 @@
   <!-- <mesh filename="package://my_egg_sensor_desc/meshes/egg_50cm_1600.stl"/> -->
 	<!-- <mesh filename="package://iiwa_tool_description/meshes/visual/tool.stl"/> -->
-		<cylinder length="0.2550" radius="0.020"/>
+		<cylinder length="0.23" radius="0.020"/>
       </geometry>
       <material name="Grey"/>

Commit message: final sync before commenting

File: src/iiwa_stack_examples/iiwa_tool/iiwa_tool_description/urdf/iiwa14_tool.urdf.xacro (robot description, xacro)
@@ -27,6 +27,6 @@
   <!-- Tool properties -->
   <property name="tool_mass" value="0.200" />
-  <property name="tool_joint_offset" value="0.00 0.00 0.00" />
-  <property name="tool_link_offset" value="0.00 0.00 0.1275" />
+  <property name="tool_joint_offset" value="0.00 0.00 0.125" />
+  <property name="tool_link_offset" value="0.00 0.00 0.125" />
   <!--  Here we define a dummy joint between the tip of the iiwa14 and the base of the tool.
   There is no offset between the two, that means the tool is attached at the robot flange ${PI/2.0} . -->
@@ -44,5 +44,6 @@
   <!-- <mesh filename="package://my_egg_sensor_desc/meshes/egg_50cm_1600.stl"/> -->
 	<!-- <mesh filename="package://iiwa_tool_description/meshes/visual/tool.stl"/> -->
-		<cylinder length="0.23" radius="0.020"/>
+		<cylinder length="0.250" radius="0.07"/>
+    <!-- <cylinder length="0.250" radius="0.001"/> -->
       </geometry>
       <material name="Grey"/>
@@ -53,5 +54,6 @@
   <!-- <mesh filename="package://my_egg_sensor_desc/meshes/egg_50cm_1600.stl"/> -->
 	<!-- <mesh filename="package://iiwa_tool_description/meshes/visual/tool.stl"/> -->
-		<cylinder length="0.23" radius="0.020"/>
+		<cylinder length="0.250" radius="0.07"/>
+    <!-- <cylinder length="0.250" radius="0.001"/> -->
       </geometry>
       <material name="Grey"/>

File: src/my_egg_sensor_desc/urdf/robot.urdf (robot description, URDF)
Before this commit: robot egg, 1 links, 0 joints
Links:
- link workpeice_link: geometry collision mesh filename=package://my_egg_sensor_desc/meshes/trash_can.stl; visual mesh filename=package://my_egg_sensor_desc/meshes/trash_can.stl
